File: board/Arduino Nano2.brd (EAGLE design)
At the start: 17.8 x 77.5 mm, 17 parts, among them J1 HEAD15-NOSS, J2 HEAD15-NOSS-1, Q1 SPD30P06PTO252

Commit message: finalized design minus silk screen
Connections:
- removed net N$13: JP2.3, JP2.4
- net N$17: now also JP2.3, JP2.4; no longer JP2.1
Routing:
- net N$4: track 0.00 -> 103.0 mm
- net N$1: track 0.00 -> 74.7 mm, vias 0 -> 2
- net D11/MOSI: track 0.00 -> 39.7 mm
- net RESET: track 0.00 -> 29.8 mm
- net GND: track 0.00 -> 24.8 mm, vias 0 -> 1
- net N$17: track 0.00 -> 10.3 mm
- net N$11: track 0.00 -> 8.58 mm
- net N$9: track 0.00 -> 7.42 mm
- net N$7: track 0.00 -> 5.39 mm
- net D4: track 0.00 -> 5.33 mm
- net N$8: track 0.00 -> 5.23 mm
- net N$10: track 0.00 -> 5.19 mm
- net N$6: track 0.00 -> 4.97 mm
- net N$12: track 0.00 -> 4.48 mm
- added copper zone on layer 16, net GND
- added copper zone on layer 1, net N$4
- removed copper zone on layer 1, net COM
- removed copper zone on layer 16, net COM
Other:
- outline, holes or cut-outs redrawn

Commit message: added gerber and updated design for production
Parts:
- moved JP1 0.70 mm to (4.90, 20.8)
- moved JP2 0.41 mm to (4.90, 15.3)
Connections:
- removed net N$17: JP2.3, JP2.4, JP3.1
- removed net RESET: J1.3, J2.3
- new net N$13: JP2.1, JP2.4, JP3.1
Routing:
- net N$4: track 103.0 -> 66.1 mm
- net RESET: track 29.8 -> 0.00 mm
- net GND: track 24.8 -> 3.35 mm
- net N$13: track 0.00 -> 13.6 mm
- net N$17: track 10.3 -> 0.00 mm
- net N$1: track 74.7 -> 80.2 mm, vias 2 -> 0
Other:
- outline, holes or cut-outs redrawn
- board text added: "+"
- board text added: "-"
- board text added: "BATT"
- board text added: "CG RE DK DB VH - 2015"
